File: electrical/pcb_boards/2t6_competition_board/capybara_rocket/capybara_rocket.kicad_pcb (KiCad board)
At the start: 4 copper layers, 140 x 68 mm, 36 parts, among them J1 Wurth_M4_62000411622, J10 Wurth_M4_62000411622, J11 Wurth_M4_62000411622, J12 Wurth_M3_62000311622, J13 Wurth_M3_62000311622, J14 Wurth_M3_62000311622, J15 Wurth_M3_62000311622, J16 Wurth_M3_62000311622, J17 Wurth_M3_62000311622, J2 Conn_01x06_Pin, J3 Wurth_M2_62000211622, J4 Wurth_M2_62000211622, J5 Wurth_M2_62000211622, J6 Wurth_M2_62000211622, J7 Wurth_M2_62000211622, J9 Wurth_M4_62000411622, U1 WRL-11812, U10 MAX756CPA_, U11 LTC3536EMSE_PBF, U12 MP3414AGJ-Z, U13 Adafruit_BMP581, U2 4754, U3 VL53L1-SATEL, U4 NUCLEO-G431KB, U5 DS1307+, U6 NE555P, U7 25LC1024-E/P, U8 DRV8212DRLR, U9 SN74LVC1G04DBVR, Y1 AB38T-32.768KHZ

Commit message: Major CPL PCB work update
Parts:
- added C1: 10μF, Capacitor_SMD:C_0805_2012Metric_Pad1.18x1.45mm_HandSolder, F.Cu at (219.2, 116.2)
- added C2: 10μF, Capacitor_SMD:C_0805_2012Metric_Pad1.18x1.45mm_HandSolder, F.Cu at (219.2, 119.2)
- added C3: 0.1μF, Capacitor_SMD:C_0805_2012Metric_Pad1.18x1.45mm_HandSolder, F.Cu at (216.0, 93.7)
- added C4: 0.1μF, Capacitor_SMD:C_0805_2012Metric_Pad1.18x1.45mm_HandSolder, F.Cu at (216.0, 96.7)
- added C5: 0.1μF, Capacitor_SMD:C_0805_2012Metric_Pad1.18x1.45mm_HandSolder, F.Cu at (216.0, 99.7)
- added C6: 0.1μF, Capacitor_SMD:C_0805_2012Metric_Pad1.18x1.45mm_HandSolder, F.Cu at (216.0, 102.7)
- added C7: 0.1μF, Capacitor_SMD:C_0805_2012Metric_Pad1.18x1.45mm_HandSolder, F.Cu at (216.0, 105.7)
- added C8: 0.1μF, Capacitor_SMD:C_0805_2012Metric_Pad1.18x1.45mm_HandSolder, F.Cu at (216.0, 108.8)
- added R1: 10Ω, Resistor_SMD:R_0603_1608Metric_Pad0.98x0.95mm_HandSolder, F.Cu at (214.6, 116.0)
- added R2: 220Ω, Resistor_SMD:R_0603_1608Metric_Pad0.98x0.95mm_HandSolder, F.Cu at (214.6, 118.5)
- added R3: 1kΩ, Resistor_SMD:R_0603_1608Metric_Pad0.98x0.95mm_HandSolder, F.Cu at (214.6, 121.0)
- added R4: 10Ω, Resistor_SMD:R_0603_1608Metric_Pad0.98x0.95mm_HandSolder, F.Cu at (220.5, 93.5)
- J1: value Wurth_M4_62000411622 -> SparkFun MAX-M10S
- J2: value Conn_01x06_Pin -> Adafruit INA219
- U13: value Adafruit_BMP581 -> Adafruit BMP581
- U2: value 4754 -> Adafruit BNO085
- U4: value NUCLEO-G431KB -> STM32 NUCLEO-G431KB
Connections:
- BT1 pad N: unconnected-(BT1-PadN) -> GND
- BT1 pad P1: unconnected-(BT1-PadP1) -> Net-(U5-VBAT)
- BT1 pad P2: unconnected-(BT1-PadP2) -> Net-(U5-VBAT)
- BZ1 pad 1: unconnected-(BZ1-+-Pad1) -> Net-(BZ1-+)
- BZ1 pad 2: unconnected-(BZ1---Pad2) -> GND
- J2 pad 1: unconnected-(J2-Pin_1-Pad1) -> 3.3V
- J2 pad 2: unconnected-(J2-Pin_2-Pad2) -> GND
- J2 pad 3: unconnected-(J2-Pin_3-Pad3) -> SCL
- J2 pad 4: unconnected-(J2-Pin_4-Pad4) -> SDA
- J3 pad 1: unconnected-(J3-Pad1) -> Net-(J3-Pad1)
- J3 pad 2: unconnected-(J3-Pad2) -> GND
- J4 pad 1: unconnected-(J4-Pad1) -> 5V
- J4 pad 2: unconnected-(J4-Pad2) -> GND
- J5 pad 1: unconnected-(J5-Pad1) -> 5V
- J5 pad 2: unconnected-(J5-Pad2) -> GND
- U1 pad JP5_10: unconnected-(U1-3.3V-PadJP5_10) -> 3.3V
- U1 pad JP5_8: unconnected-(U1-DIN-PadJP5_8) -> XBEE_TX
- U1 pad JP5_9: unconnected-(U1-DOUT-PadJP5_9) -> XBEE_RX
- U13 pad 1: unconnected-(U13-VCC-Pad1) -> 3.3V
- U13 pad 2: unconnected-(U13-GND-Pad2) -> GND
- U13 pad 3: unconnected-(U13-SCL-Pad3) -> SCL
- U13 pad 4: unconnected-(U13-SDA-Pad4) -> SDA
- U2 pad JP1_1: unconnected-(U2-VIN-PadJP1_1) -> 3.3V
- U2 pad JP1_3: unconnected-(U2-GND-PadJP1_3) -> GND
- U2 pad JP1_4: unconnected-(U2-SCL-PadJP1_4) -> SCLK
- U2 pad JP1_5: unconnected-(U2-SDA-PadJP1_5) -> MISO
- U2 pad JP2_5: unconnected-(U2-DI-PadJP2_5) -> MOSI
- U2 pad JP2_6: unconnected-(U2-CS-PadJP2_6) -> CS
- U3 pad 2: unconnected-(U3-SCL_I-Pad2) -> SCL
- U3 pad 4: unconnected-(U3-SDA_I-Pad4) -> SDA
- U4 pad CN3_6: unconnected-(U4-PA7(A6)-PadCN3_6) -> MOSI
- U4 pad CN3_7: unconnected-(U4-PA6/PA15(A5)-PadCN3_7) -> MISO
- U4 pad CN3_8: unconnected-(U4-PA5/PB7(A4)-PadCN3_8) -> SCLK
- U4 pad CN3_9: unconnected-(U4-PA4(A3)-PadCN3_9) -> CS
- U4 pad CN4_1: unconnected-(U4-PA9(D1)-PadCN4_1) -> XBEE_TX
- U4 pad CN4_2: unconnected-(U4-PA10(D0)-PadCN4_2) -> XBEE_RX
- U4 pad CN4_7: unconnected-(U4-PB7(D4)-PadCN4_7) -> SDA
- U4 pad CN4_8: unconnected-(U4-PA15(D5)-PadCN4_8) -> SCL
- U5 pad 1: unconnected-(U5-X1-Pad1) -> X1
- U5 pad 2: unconnected-(U5-X2-Pad2) -> X2
- U5 pad 3: unconnected-(U5-VBAT-Pad3) -> Net-(U5-VBAT)
- U5 pad 4: unconnected-(U5-GND-Pad4) -> GND
- U5 pad 5: unconnected-(U5-SDA-Pad5) -> SDA
- U5 pad 6: unconnected-(U5-SCL-Pad6) -> SCL
- U5 pad 8: unconnected-(U5-VCC-Pad8) -> 5V
- U6 pad 1: unconnected-(U6-GND-Pad1) -> GND
- U6 pad 2: unconnected-(U6-TRIG-Pad2) -> Net-(U6-THRES)
- U6 pad 3: unconnected-(U6-OUT-Pad3) -> Net-(U6-OUT)
- U6 pad 4: unconnected-(U6-~{RST}-Pad4) -> 5V
- U6 pad 5: unconnected-(U6-CONT-Pad5) -> Net-(U6-CONT)
- U6 pad 6: unconnected-(U6-THRES-Pad6) -> Net-(U6-THRES)
- U6 pad 7: unconnected-(U6-DISCH-Pad7) -> Net-(U6-DISCH)
- U6 pad 8: unconnected-(U6-VCC-Pad8) -> 5V
- Y1 pad 1: unconnected-(Y1-Pad1) -> X1
- Y1 pad 2: unconnected-(Y1-Pad2) -> X2
Other:
- board size 140 x 68 mm -> 145 x 65 mm
