File: electrical/pcb_boards/2t6_competition_board/capybara_rocket/_autosave-capybara_rocket.kicad_pcb (KiCad board)
At the start: 4 copper layers, 145 x 65 mm, 51 parts, among them J1 SparkFun MAX-M10S, J10 Wurth_M4_62000411622, J11 Wurth_M4_62000411622, J12 Wurth_M3_62000311622, J13 Wurth_M3_62000311622, J14 Wurth_M3_62000311622, J15 Wurth_M3_62000311622, J16 Wurth_M3_62000311622, J17 Wurth_M3_62000311622, J3 Wurth_M2_62000211622, J4 Wurth_M2_62000211622, J5 Wurth_M2_62000211622, J6 Wurth_M2_62000211622, J7 Wurth_M2_62000211622, J9 Wurth_M4_62000411622, U1 WRL-11812, U10 MAX756CPA_, U11 LTC3536EMSE_PBF, U12 MP3414AGJ-Z, U13 Adafruit BMP581, U14 INA219BIDR, U2 Adafruit BNO085, U3 VL53L1-SATEL, U4 STM32 NUCLEO-G431KB, U5 DS1307+, U6 NE555P, U7 25LC1024-E/P, U8 DRV8212DRLR, U9 SN74LVC1G04DBVR, Y1 AB38T-32.768KHZ

Commit message: March 8th updates
Parts:
- removed U3: VL53L1-SATEL, RSX_CanSat_Custom_KiCad_Footprints:J_Wurth_WR-WTB_62000411622
- added D1: LED, DigiKey:WL-SMCW_0603, F.Cu at (162.4, 84.5)
- added D2: LED, DigiKey:WL-SMCW_0603, F.Cu at (162.4, 87.0)
- added D3: LED, DigiKey:WL-SMCW_0603, F.Cu at (162.4, 89.5)
- added D4: LED, DigiKey:WL-SMCW_0603, F.Cu at (162.4, 92.0)
- added D5: LED, DigiKey:WL-SMCW_0603, F.Cu at (162.4, 94.5)
- added J2: VL53L1-SATEL, RSX_CanSat_Custom_KiCad_Footprints:J_Wurth_WR-WTB_62000411622, F.Cu at (126.5, 137.8)
- BZ1: footprint Buzzer_Beeper:Buzzer_12x9.5RM7.6 -> RSX_CanSat_Custom_KiCad_Footprints:Buzzer_12x9.5RM7.6
- U10: footprint RSX_CanSat_Custom_KiCad_Footprints:DIP794W47P254L991H457Q8 -> Package_DIP:DIP-8_W7.62mm
- U7: footprint RSX_CanSat_Custom_KiCad_Footprints:PDIP8_300MC_MCH -> Package_DIP:DIP-8_W7.62mm
- moved U10 5.24 mm to (170.0, 111.5)
- moved U7 0.06 mm to (180.6, 111.3)
Connections:
- net Net-(U14-VIN+) renamed 3.6V
- C5 pad 1: GND -> 3.3V
- C5 pad 2: 3.3V -> GND
- U13 pad 5: Net-(U13-PadVIN-) -> unconnected-(U13-PadVIN-)
- U13 pad 6: Net-(U13-PadVIN+) -> unconnected-(U13-PadVIN+)
- U4 pad CN3_11: unconnected-(U4-WING_PWM(PA1(A1))-PadCN3_11) -> WING_PWM
- U4 pad CN3_12: unconnected-(U4-WING_DIR(PA0(A0))-PadCN3_12) -> WING_DIR
- U4 pad CN4_10: unconnected-(U4-G_CAM_OUT(PF0(D7))-PadCN4_10) -> G_CAM_OUT
- U4 pad CN4_11: unconnected-(U4-PG_CAM_OUT(PF1(D8))-PadCN4_11) -> PG_CAM_OUT
- U4 pad CN4_12: unconnected-(U4-PG_CAM_IN(PA8(D9))-PadCN4_12) -> PG_CAM_IN
- U4 pad CN4_13: unconnected-(U4-CC_REL(PA11(D10))-PadCN4_13) -> CC_REL
- U4 pad CN4_14: unconnected-(U4-AILERON(PB5(D11))-PadCN4_14) -> AILERON
- U4 pad CN4_15: unconnected-(U4-ELEVATOR(PB4(D12))-PadCN4_15) -> ELEVATOR
- U4 pad CN4_4: unconnected-(U4-GND_CN4-PadCN4_4) -> GND
- U4 pad CN4_5: unconnected-(U4-NC_REL(PA12(D2))-PadCN4_5) -> NC_REL
- U4 pad CN4_6: unconnected-(U4-EGG_REL(PB0(D3))-PadCN4_6) -> EGG_REL
- U4 pad CN4_9: unconnected-(U4-G_CAM_IN(PB6(D6))-PadCN4_9) -> G_CAM_IN
