File: electrical/pcb_boards/2t6_competition_boards/capybara_rocket/capybara_rocket.kicad_pcb (KiCad board)
At the start: 4 copper layers, 160 x 65 mm, 157 parts, among them J1 3.6V Battery, J10 Elevator, J11 SparkFun MAX-M10S, J12 Aileron 1, J13 Aileron 2, J14 Ground Camera, J15 Payload Camera, J16 DC Motor, J2 1.2V Battery, J3 3.6V Switch, J4 1.2V Switch, J5 LED, J6 NC, J7 CC, J8 VL53L1-SATEL, J9 Egg, Q1 SI4435DDY, Q2 SI4435DDY, U1 DS1307+, U10 TPS3839, U11 MP3414, U12 SN74LVC1G04, U13 MCP1640, U14 TPS3839, U15 STM32 NUCLEO-G431KB, U16 SN74AUP1G04, U17 SparkFun XBee Explorer, U2 Adafruit BNO085, U3 TLC555, U4 EEPROM, U5 LTC3536, U6 LTC3536, U7 Adafruit BMP581, U8 DRV8212, U9 INA219, Y1 AB38T-32.768KHZ

Commit message: All fixes made on CPL board except inductor change for LTC353:
Parts:
- added C10: 0.1μF, Capacitor_SMD:C_0805_2012Metric_Pad1.18x1.45mm_HandSolder, F.Cu at (108.5, 79.4)
- added C19: 0.1μF, Capacitor_SMD:C_0805_2012Metric_Pad1.18x1.45mm_HandSolder, F.Cu at (90.2, 85.2)
- added C20: 0.1μF, Capacitor_SMD:C_0805_2012Metric_Pad1.18x1.45mm_HandSolder, F.Cu at (188.4, 122.0)
- added C21: 10μF, Capacitor_SMD:C_1206_3216Metric_Pad1.33x1.80mm_HandSolder, F.Cu at (83.4, 83.0)
- added C23: 0.1μF, Capacitor_SMD:C_0805_2012Metric_Pad1.18x1.45mm_HandSolder, F.Cu at (188.4, 118.0)
- added C27: 0.1μF, Capacitor_SMD:C_0805_2012Metric_Pad1.18x1.45mm_HandSolder, F.Cu at (188.4, 76.2)
- added C29: 0.1μF, Capacitor_SMD:C_0805_2012Metric_Pad1.18x1.45mm_HandSolder, F.Cu at (188.4, 72.1)
- added G***: LOGO, RSX_CanSat_Graphics:maple_leaf, F.Cu at (205.2, 128.2)
- added L1: 4.7μH, RSX_CanSat_Custom_KiCad_Footprints:HPC_8040NC-4R7M, F.Cu at (239.0, 93.8)
- added L2: 4.7μH, RSX_CanSat_Custom_KiCad_Footprints:HPC_8040NC-4R7M, F.Cu at (239.6, 102.8)
- R24, R25: value 2.2kΩ -> 4.7kΩ
- moved TP1 6.00 mm to (228.2, 113.5)
- moved TP2 6.00 mm to (228.2, 107.5)
- moved U10 0.63 mm to (184.2, 122.2)
- moved U12 0.63 mm to (184.2, 117.8)
- moved U16 0.63 mm to (184.2, 72.0)
- moved U14 0.63 mm to (184.2, 76.4)
- turned U8 to 0 degrees
- renumbered C10 to C11, C11 to C12, C12 to C13, C13 to C14, C14 to C15, C15 to C16, C16 to C17, C17 to C18, C18 to C22, C19 to C24, C20 to C25, C21 to C26, C22 to C28, TP2 to TP1, TP1 to TP2
Connections:
- J1 pad 2: 3.6V B -> 3.6V BT
- J10 pad 2: ELEVATOR -> 5.5V
- J10 pad 3: 5.5V -> ELEVATOR
- J12 pad 2: AILERON -> 5.5V
- J12 pad 3: 5.5V -> AILERON
- J13 pad 2: AILERON -> 5.5V
- J13 pad 3: 5.5V -> AILERON
- J14 pad 2: G_CAM_IN -> 5.5V
- J14 pad 3: G_CAM_OUT -> G_CAM_IN
- J14 pad 4: 5.5V -> G_CAM_OUT
- J15 pad 2: PG_CAM_IN -> 5.5V
- J15 pad 3: PG_CAM_OUT -> PG_CAM_IN
- J15 pad 4: 5.5V -> PG_CAM_OUT
- J2 pad 2: 1.2V B -> 1.2V BT
- J3 pad 1: GND -> 3.6V BT
- J4 pad 1: GND -> 1.2V BT
- J6 pad 2: NC_REL -> 5.5V
- J6 pad 3: 5.5V -> NC_REL
- J7 pad 2: CC_REL -> 5.5V
- J7 pad 3: 5.5V -> CC_REL
- J8 pad 2: SDA -> 3.3V
- J8 pad 3: SCL -> SDA
- J8 pad 4: 3.3V -> SCL
- J9 pad 2: EGG_REL -> 5.5V
- J9 pad 3: 5.5V -> EGG_REL
- Q1 pad 2: unconnected-(Q1-Pad2) -> 3.6V B
- Q1 pad 3: unconnected-(Q1-Pad3) -> 3.6V B
- Q1 pad 6: unconnected-(Q1-Pad6) -> 3.6V+
- Q1 pad 7: unconnected-(Q1-Pad7) -> 3.6V+
- Q1 pad 8: unconnected-(Q1-Pad8) -> 3.6V+
- Q2 pad 2: unconnected-(Q2-Pad2) -> 1.2V B
- Q2 pad 3: unconnected-(Q2-Pad3) -> 1.2V B
- Q2 pad 6: unconnected-(Q2-Pad6) -> 1.2V
- Q2 pad 7: unconnected-(Q2-Pad7) -> 1.2V
- Q2 pad 8: unconnected-(Q2-Pad8) -> 1.2V
- TP1 pad 1: 1.2V -> 1.2V B
- TP2 pad 1: 1.2V B -> 1.2V
- U15 pad CN3_1: 3.3V MCU -> unconnected-(U15-VIN-PadCN3_1)
- U15 pad CN3_14: unconnected-(U15-3V3-PadCN3_14) -> 3.3V MCU
- U15 pad CN3_15: unconnected-(U15-T_SWO(PB3/PB8(D13))-PadCN3_15) -> IMU_INT
- U2 pad JP1_6: unconnected-(U2-~{INT}-PadJP1_6) -> IMU_INT
- U2 pad JP2_2: unconnected-(U2-P0-PadJP2_2) -> GND
- U2 pad JP2_3: unconnected-(U2-P1-PadJP2_3) -> GND
- U2 pad JP2_4: unconnected-(U2-~{RST}-PadJP2_4) -> 3.3V
- U2 pad JP2_5: unconnected-(U2-DI-PadJP2_5) -> GND
- U2 pad JP2_6: unconnected-(U2-CS-PadJP2_6) -> 3.3V
- U4 pad 3: GND -> 3.3V
- U5 pad 13: unconnected-(U5-EPAD-Pad13) -> GND
- U5 pad 3: unconnected-(U5-MODE/SYNC-Pad3) -> GND
- U6 pad 13: unconnected-(U6-EPAD-Pad13) -> GND
- U6 pad 3: unconnected-(U6-MODE/SYNC-Pad3) -> GND
- U9 pad 1: unconnected-(U9-A1-Pad1) -> GND
- U9 pad 2: unconnected-(U9-A0-Pad2) -> GND
Routing:
- net 3.3V: track 312.0 -> 354.6 mm, vias 11 -> 13
- net 3.3V MCU: track 105.4 -> 132.9 mm
- net IMU_INT: track 0.00 -> 23.4 mm
- net GND: track 83.5 -> 100.2 mm
- net 3.6V BT: track 0.00 -> 10.8 mm
- net INV_PWM_1: track 50.1 -> 59.1 mm
- net 5.5V: track 347.8 -> 339.5 mm, vias 7 -> 6
- net INV_PWM_2: track 51.2 -> 58.0 mm
- net 1.2V BT: track 0.00 -> 5.60 mm
- net 1.2V B: track 99.0 -> 104.2 mm, vias 4 -> 5
- net 3.6V B: track 86.9 -> 91.6 mm, vias 3 -> 4
- net DC_PWM_2: track 5.05 -> 9.56 mm, vias 0 -> 1
- net 3.6V+: track 83.5 -> 87.5 mm
- net 1.2V: track 66.7 -> 70.5 mm
- net AILERON: track 130.2 -> 127.1 mm
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Other:
- board text added: "4.7kΩ"
- board text removed: "2.2kΩ"

Commit message: V2 of CPL board
Parts:
- removed the G*** at (208.6, 97.8)
- removed the G*** at (152.3, 127.2)
- removed the L1 at (215.7, 97.0)
- removed the L2 at (201.5, 98.5)
- added G***: LOGO, LOGO, F.Cu at (100.6, 93.4)
- added G***: LOGO, LOGO, F.Cu at (165.4, 81.2)
- added G***: LOGO, LOGO, F.Cu at (146.0, 93.0)
- added G***: LOGO, LOGO, F.Cu at (146.0, 123.0)
- added G***: LOGO, LOGO, B.Cu at (213.2, 128.2)
- added G***: LOGO, LOGO, B.Cu at (86.6, 89.6)
- added G***: LOGO, LOGO, F.Cu at (123.0, 107.4)
- added G***: LOGO, RSX_CanSat_Graphics:uoft_eng_logo, B.Cu at (153.0, 127.4)
- added G***: LOGO, RSX_CanSat_Graphics:music, F.Cu at (162.2, 121.2)
- added G***: LOGO, LOGO, F.Cu at (123.0, 86.4)
- added G***: LOGO, LOGO, F.Cu at (187.4, 100.0)
- moved L2 36.3 mm to (203.4, 99.6)
- moved L1 25.3 mm to (213.8, 95.9)
- moved U6 1.52 mm to (204.8, 107.0)
- moved U5 1.52 mm to (212.4, 88.5)
- moved C17 0.86 mm to (216.5, 84.7)
- moved C18 0.86 mm to (200.7, 110.8)
- moved G*** 0.68 mm to (163.2, 77.4)
- moved G*** 0.63 mm to (224.4, 79.8), turned to 90 degrees
- turned G*** to 90 degrees (x2)
Routing:
- net 3.3V: track 354.6 -> 359.7 mm, vias 13 -> 12
- net Net-(U5-VC): track 3.36 -> 4.87 mm
- net Net-(U6-VC): track 3.36 -> 4.87 mm
- net 3.3V MCU: track 132.9 -> 134.1 mm
- net MOSI: track 54.9 -> 55.9 mm
- net 3.6V-: track 135.8 -> 134.8 mm, vias 14 -> 12
- net GND: track 100.2 -> 99.3 mm, vias 32 -> 34
- net 5.5V: vias 6 -> 7
Other:
- board text added: "B82462G4"
- board text added: "HPC 8040NC"
- board text added: "SRN6045"
- board text added: "SW_IN"
- board text added: "SW_OUT"
- board text removed: "15μH"
