File: electrical/pcb_boards/2t6_competition_boards/capybara_rocket/capybara_rocket.kicad_sch (KiCad schematic)
At the start: 117 parts, among them J1 3.6V Battery, J10 Elevator, J11 SparkFun MAX-M10S, J12 Aileron 1, J13 Aileron 2, J14 Ground Camera, J15 Payload Camera, J16 DC Motor, J2 1.2V Battery, J3 3.6V Switch, J4 1.2V Switch, J5 LED, J6 NC, J7 CC, J8 VL53L1-SATEL, J9 Egg, Q1 SI4435DDY, Q2 SI4435DDY, U1 DS1307+, U10 TPS3839, U11 MP3414, U12 SN74LVC1G04, U13 MCP1640, U14 TPS3839, U15 STM32 NUCLEO-G431KB, U16 SN74AUP1G04, U17 SparkFun XBee Explorer, U2 Adafruit BNO085, U3 TLC555, U4 EEPROM, U5 LTC3536, U6 LTC3536, U7 Adafruit BMP581, U8 DRV8212, U9 INA219, Y1 AB38T-32.768KHZ

Commit message: Halfway through schematic fixes
Parts:
- R14, R15, R16, R17, R19, R20, R21, R22: value 1kΩ -> 100Ω
- R18: value 1.5kΩ -> 100Ω
Connections:
- net 1.2V B: now also C29.2; no longer C29.1
- net 3.6V B: now also C28.2; no longer C28.1
- net AILERON: now also J12.3, J13.3; no longer J12.1, J13.1
- net CC_REL: now also J7.3; no longer J7.1
- net EGG_REL: now also J9.3; no longer J9.1
- net ELEVATOR: now also J10.3; no longer J10.1
- net GND: now also C28.1, C29.1, J10.1, J12.1, J13.1, J6.1, J7.1, J9.1; no longer C28.2, C29.2, J10.3, J12.3, J13.3, J6.3, J7.3, J9.3
- net NC_REL: now also J6.3; no longer J6.1
Other:
- moved on the sheet: C27, C28, D2, D6, D7, Q1, R15, R19, R20, TP1, TP10, TP2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

Commit message: All fixes made on CPL board except inductor change for LTC353:
Parts:
- removed C25: 0.1μF, Capacitor_SMD:C_0805_2012Metric_Pad1.18x1.45mm_HandSolder, symbol Device:C
- removed L1, L2: 15μH, RSX_CanSat_Custom_KiCad_Footprints:WE-TPC_4828, symbol RSX_CanSat_Custom_KiCad_Symbols:WE-TPC_4828
- added C10: 0.1μF, Capacitor_SMD:C_0805_2012Metric_Pad1.18x1.45mm_HandSolder, symbol Device:C
- added L1, L2: 4.7μH, RSX_CanSat_Custom_KiCad_Footprints:HPC_8040NC-4R7M, symbol Device:L
- renumbered C10 to C11, C11 to C12, C12 to C13, C13 to C14, C14 to C15, C15 to C16, C16 to C17, C17 to C18, C23 to C19, C27 to C20, C24 to C21, C18 to C22, C28 to C23, C19 to C24, C20 to C25, C21 to C26, C26 to C27, C22 to C28, D2 to D1, D1 to D2, R15 to R14, R14 to R15, TP2 to TP1, TP1 to TP2
Connections:
- net 1.2V: now also R15.2, TP2.1; no longer R14.2, TP1.1
- net 1.2V B: now also R14.2, TP1.1; no longer J2.2, J4.1, R15.2, TP2.1
- net 3.3V: now also C8.1, J8.2, C10.2; no longer J8.3
- net 3.6V B: no longer J1.2, J3.1
- net 5.5V: now also J14.2, J15.2; no longer J14.3, J15.3
- net GND: now also J14.1, J15.1, J8.1, C10.1; no longer C8.1, J14.4, J15.4, J8.4
- net G_CAM_IN: now also J14.3; no longer J14.2
- net G_CAM_OUT: now also J14.4; no longer J14.1
- net PG_CAM_IN: now also J15.3; no longer J15.2
- net PG_CAM_OUT: now also J15.4; no longer J15.1
- net SCL: now also J8.4; no longer J8.1
- net SDA: now also J8.3; no longer J8.2
- net at U6.4 (SW1): now also L2.1
- net at U6.6 (SW2): now also L2.2
- net at U5.4 (SW1): now also L1.1
- net at U5.6 (SW2): now also L1.2
- net INT renamed IMU_INT
- new net 1.2V BT: J2.2, J4.1
- new net 3.6V BT: J1.2, J3.1
Other:
- note added: "Test Point Circuits"
- note removed: "LED Indicator Circuits"
- note removed: "change the 15uH VOTH ltc3536 inductors to"
- note removed: "https://www.digikey.ca/en/products/detail/tai-tech-advanced-electronics-co-ltd/HPC-8040NC-4R7M/17835630"
- moved on the sheet: C16, C19, C21, C22, C4, J1, J14, J15, J16, J2, J3, J4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
