File: electrical/pcb_boards/2t6_competition_boards/capybara_habitat/capybara_habitat.kicad_pcb (KiCad board)
At the start: 2 copper layers, 137.3 x 78 mm, 120 parts, among them J1 Barrel_Jack, J10 monitor2_power, J11 aud_sig_out_a, J12 spare_usb_2nd_disp_pwr, J13 2nd_disp_sw, J14 spkrs_sw, J15 Raspberry_Pi_4, J16 Raspberry_Pi_4, J17 charger_buck_in, J2 leds_power, J3 monitor1_power, J4 charger_buck_in, J5 leds_sw, J6 1st_disp_sw, J7 aud_sig_out_b, J8 vbatt, J9 aud_sig_in, U1 TPS22810DBV, U2 TPS22810DBV, U3 TPS22810DBV, U4 Adafruit_INA219, U5 Adafruit_INA219, U6 PAM8406D, U7 TPS22810DBV, U8 LT8610ABEMSE-5-TRPBF, U9 LTC3114IFE-1_TRPBF

Commit message: Fixed gerber
Parts:
- moved G*** 1.14 mm to (120.5, 126.5)
Changed lines of the file:
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@@
 	(footprint "RSX_CanSat_Graphics:capybara"
 		(layer "F.Cu")
-		(at 121.4 125.875143)
+		(at 120.453515 126.505143)
 		(property "Reference" "G***"
 			(at 0 0 0)
